File: steering_wheel_shield_2019.sch (KiCad schematic (older format))
At the start: 6 parts

Commit message: can transceiver and more mcu connections
Parts:
- added C?: 0.1uF, Capacitor_SMD:C_0603_1608Metric_Pad1.05x0.95mm_HandSolder, symbol Device:CP
- added C?: 4.7nF, Capacitor_SMD:C_0603_1608Metric_Pad1.05x0.95mm_HandSolder, symbol Device:C
- added C?: 0.1uF, symbol Device:C
- added J?: VEHICLE, symbol Connector_Generic:Conn_01x06
- added J?: DEBUG, symbol Connector_Generic:Conn_01x07
- added JP?: CAN_TERM, Connector_PinHeader_2.54mm:PinHeader_1x03_P2.54mm_Vertical, symbol Jumper:Jumper_3_Open
- added R? (x2): 60, Resistor_SMD:R_0805_2012Metric_Pad1.15x1.40mm_HandSolder, symbol Device:R_US
- added U?: SN65HVD232, Package_SO:SOIC-8_3.9x4.9mm_P1.27mm, symbol Interface_CAN_LIN:SN65HVD232
Connections:
- net labels added: 5V, CANH, CANL, CAN_RX, CAN_TX, NRST, SWCLK, SWDIO, SWO, VIN
- wire segments 20 -> 74
- no-connect marks 0 -> 1
Other:
- moved on the sheet: U?

Commit message: mcu in progress; drc mostly passes
Parts:
- added C1, C3, C4, C5, C6, C7: 0.1uF, symbol Device:C
- C11: renamed from C?; value C -> 10uF
- C9: renamed from C?; value C -> 22uF
- gave numbers to parts that had none: 13
Connections:
- wire segments 74 -> 113
Other:
- moved on the sheet: C2, U1

Commit message: power circuitry; mcu gpio pins; oscillator
Parts:
- added C? (x2): 26pF, symbol Device:C
- added D? (x2): B340A-13-F, digikey-footprints:DO-214AC, symbol dk_Diodes-Rectifiers-Single:B340A-13-F
- added Y?: Crystal, symbol Device:Crystal
Connections:
- net labels added: PA0, PA1, PA10, PA15, PA2, PA3, PA4, PA5, PA6, PA7, PA8, PA9, PB0, PB1, PB10, PB11, PB12, PB13, PB14, PB15, PB2, PB4, PB5, PB6, PB7, PB8, PB9, PC0, PC1, PC10, PC11, PC12, PC13, PC14, PC15, PC2, PC3, PC4, PC5, PC6, PC7, PC8, PC9
- wire segments 113 -> 177
Other:
- moved on the sheet: J1

Commit message: led indicator
Parts:
- added D?: LED, symbol Device:LED
- added R?: 68, symbol Device:R_US
Connections:
- wire segments 177 -> 182
Other:
- moved on the sheet: C?, Y?
Changed lines of the file:
@@
 	6800 1400 6800 1200
 Connection ~ 6800 1200
-Wire Wire Line
-	2150 4000 2150 4200
-Wire Wire Line
-	2150 4200 2450 4200
-Wire Wire Line
-	2150 4300 2450 4300
-Wire Wire Line
-	2150 4500 2150 4300
-Connection ~ 1700 4000
-Wire Wire Line
-	1700 4000 2150 4000
-Connection ~ 1700 4500
-Wire Wire Line
-	1700 4500 2150 4500
-Wire Wire Line
-	1700 4500 1700 4400
-Wire Wire Line
-	1500 4500 1700 4500
-Wire Wire Line
-	1700 4000 1700 4100
-Wire Wire Line
-	1500 4000 1700 4000
-Connection ~ 1100 4250
-Wire Wire Line
-	1100 4500 1200 4500
-Wire Wire Line
-	1100 4250 1100 4500
-Wire Wire Line
-	1100 4250 1000 4250
-Wire Wire Line
-	1100 4000 1100 4250
-Wire Wire Line
-	1200 4000 1100 4000
-Text GLabel 1000 4250 0    50   Input ~ 0
+Connection ~ 1450 3650
+Connection ~ 1450 4150
+Wire Wire Line
+	1450 4150 1450 4050
+Wire Wire Line
+	1250 4150 1450 4150
+Wire Wire Line
+	1450 3650 1450 3750
+Wire Wire Line
+	1250 3650 1450 3650
+Connection ~ 850  3900
+Wire Wire Line
+	850  4150 950  4150
+Wire Wire Line
+	850  3900 850  4150
+Wire Wire Line
+	850  3900 750  3900
+Wire Wire Line
+	850  3650 850  3900
+Wire Wire Line
+	950  3650 850  3650
+Text GLabel 750  3900 0    50   Input ~ 0
 GND
 $Comp
 L Device:C C?
 U 1 1 5DA26385
-P 1350 4000
-F 0 "C?" V 1098 4000 50  0000 C CNN
-F 1 "26pF" V 1189 4000 50  0000 C CNN
-F 2 "" H 1388 3850 50  0001 C CNN
-F 3 "~" H 1350 4000 50  0001 C CNN
-	1    1350 4000
+P 1100 3650
+F 0 "C?" V 848 3650 50  0000 C CNN
+F 1 "26pF" V 939 3650 50  0000 C CNN
+F 2 "" H 1138 3500 50  0001 C CNN
+F 3 "~" H 1100 3650 50  0001 C CNN
+	1    1100 3650
 	0    1    1    0
 $EndComp
@@
 L Device:Crystal Y?
 U 1 1 5DA251CF
-P 1700 4250
-F 0 "Y?" V 1654 4381 50  0000 L CNN
-F 1 "Crystal" V 1745 4381 50  0000 L CNN
-F 2 "" H 1700 4250 50  0001 C CNN
-F 3 "~" H 1700 4250 50  0001 C CNN
-	1    1700 4250
+P 1450 3900
+F 0 "Y?" V 1404 4031 50  0000 L CNN
+F 1 "Crystal" V 1495 4031 50  0000 L CNN
+F 2 "" H 1450 3900 50  0001 C CNN
+F 3 "~" H 1450 3900 50  0001 C CNN
+	1    1450 3900
 	0    1    1    0
 $EndComp
@@
 L Device:C C?
 U 1 1 5DA26E1E
-P 1350 4500
-F 0 "C?" V 1098 4500 50  0000 C CNN
-F 1 "26pF" V 1189 4500 50  0000 C CNN
-F 2 "" H 1388 4350 50  0001 C CNN
-F 3 "~" H 1350 4500 50  0001 C CNN
-	1    1350 4500
+P 1100 4150
+F 0 "C?" V 848 4150 50  0000 C CNN
+F 1 "26pF" V 939 4150 50  0000 C CNN
+F 2 "" H 1138 4000 50  0001 C CNN
+F 3 "~" H 1100 4150 50  0001 C CNN
+	1    1100 4150
 	0    1    1    0
 $EndComp
@@
 Wire Wire Line
 	3850 6100 3950 6100
+$Comp
+L Device:LED D?
+U 1 1 5DCB5BA5
+P 1700 4600
+F 0 "D?" H 1700 4700 50  0000 C CNN
+F 1 "LED" H 1700 4800 50  0000 C CNN
+F 2 "" H 1700 4600 50  0001 C CNN
+F 3 "~" H 1700 4600 50  0001 C CNN
+	1    1700 4600
+	-1   0    0    1
+$EndComp
+Wire Wire Line
+	2450 4300 2250 4300
+Wire Wire Line
+	2250 4300 2250 4150
+Wire Wire Line
+	1450 4150 2250 4150
+Wire Wire Line
+	2450 4200 2350 4200
+Wire Wire Line
+	2350 4200 2350 3650
+Wire Wire Line
+	1450 3650 2350 3650
+Wire Wire Line
+	1850 4600 1950 4600
+Wire Wire Line
+	1950 4600 1950 4400
+Wire Wire Line
+	1950 4400 2450 4400
+Wire Wire Line
+	1450 4600 1550 4600
+Text GLabel 1050 4600 0    50   Input ~ 0
+3V3
+Wire Wire Line
+	1050 4600 1150 4600
+$Comp
+L Device:R_US R?
+U 1 1 5DCF4306
+P 1300 4600
+F 0 "R?" V 1505 4600 50  0000 C CNN
+F 1 "68" V 1414 4600 50  0000 C CNN
+F 2 "" V 1340 4590 50  0001 C CNN
+F 3 "~" H 1300 4600 50  0001 C CNN
+	1    1300 4600
+	0    -1   -1   0
+$EndComp
 $EndSCHEMATC

Commit message: add output connects
Parts:
- added J10, J11, J3, J5, J7, J9: Conn_01x15, symbol Connector_Generic:Conn_01x15
- added J4, J6, J8: Conn_01x13, symbol Connector_Generic:Conn_01x13
- gave numbers to parts that had none: 7
Connections:
- wire segments 182 -> 397

Commit message: start layout
Parts:
- removed J2: DEBUG, symbol Connector_Generic:Conn_01x07
- added J12: ALT_PWR, Connector_BarrelJack:BarrelJack_CUI_PJ-102AH_Horizontal, symbol Connector_Generic:Conn_01x02
- added J2: DEBUG, Connector_PinSocket_2.54mm:PinSocket_2x03_P2.54mm_Vertical, symbol Connector_Generic:Conn_01x06
- C1, C11, C12, C13, C2, C3, C4, C5, C6, C7, C9, D2: footprint (none) -> Capacitor_SMD:C_0805_2012Metric_Pad1.15x1.40mm_HandSolder
- C10, C8: footprint Capacitor_SMD:C_0603_1608Metric_Pad1.05x0.95mm_HandSolder -> Capacitor_SMD:C_0805_2012Metric_Pad1.15x1.40mm_HandSolder
- D1: footprint (none) -> rahulsalvi:DO-214AB_no_polarity
- F1: footprint (none) -> Fuse:Fuse_0805_2012Metric_Pad1.15x1.40mm_HandSolder
- J1: footprint (none) -> Connector_PinSocket_2.54mm:PinSocket_1x06_P2.54mm_Vertical
- J10, J11, J3, J5, J7, J9: footprint (none) -> Connector_PinSocket_2.54mm:PinSocket_1x15_P2.54mm_Vertical
- J4, J6, J8: footprint (none) -> Connector_PinSocket_2.54mm:PinSocket_1x13_P2.54mm_Vertical
- R3: footprint (none) -> Resistor_SMD:R_0805_2012Metric_Pad1.15x1.40mm_HandSolder
- Y1: value Crystal -> 8MHz; footprint (none) -> Crystal:Crystal_SMD_HC49-SD
Connections:
- net labels added: VTref
- wire segments 397 -> 399
Other:
- moved on the sheet: C1, C10, C11, C12, C13, C2, C3, C4, C5, C6, C7, C8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
